File: sch/adapter/adapter.kicad_pcb (KiCad board)
At the start: 2 copper layers, 58 parts, among them J1 PB2, J10 PB4, J11 PB5, J12 PB6, J13 PB7, J14 PB10, J15 PB11, J16 VBAT, J17 CAN2, J18 CAN1, J19 PA0-7, J2 PH2, J20 PA8-16, J21 USART1, J22 USART2, J26 RS485, J27 PWR1, J28 PWR2, J29 POWER, J3 PH3, J4 PC13, J5 PC14, J6 PC15, J7 PB0, J8 PB1, J9 PB3, SW1 RESET, U1 AT32F435-lqfp48, U2 TJA1049T, U3 TJA1049T, U4 MAX485E, U5 AMS1117-3.3, Y1 8.0 MHz

Commit message: Preparing SilkScreen
Parts:
- removed J27: PWR1, Connector_PinHeader_2.54mm:PinHeader_1x03_P2.54mm_Vertical
- removed J28: PWR2, Connector_PinHeader_2.54mm:PinHeader_1x03_P2.54mm_Vertical
- added C11: 100n, Capacitor_SMD:C_0805_2012Metric, F.Cu at (124.0, 49.9)
- added PWR1: PWR1, Connector_PinHeader_2.54mm:PinHeader_1x03_P2.54mm_Vertical, F.Cu at (111.6, 88.9)
- added PWR2: PWR2, Connector_PinHeader_2.54mm:PinHeader_1x03_P2.54mm_Vertical, F.Cu at (114.4, 49.0)
- added U6: W25Q32JVSS, Package_SO:SOIC-8_5.23x5.23mm_P1.27mm, B.Cu at (124.6, 53.8)
- PB0: renamed from J7; value PB0 -> ~
- PB1: renamed from J8; value PB1 -> ~
- PB10: renamed from J14; value PB10 -> ~
- PB11: renamed from J15; value PB11 -> ~
- PB2: renamed from J1; value PB2 -> ~
- PB3: renamed from J9; value PB3 -> ~
- PB4: renamed from J11; value PB5 -> ~
- PB5: renamed from J10; value PB4 -> ~
- PB6: renamed from J12; value PB6 -> ~
- PB7: renamed from J13; value PB7 -> ~
- PC13: renamed from J4; value PC13 -> ~
- PC14: renamed from J5; value PC14 -> ~
- PC15: renamed from J6; value PC15 -> ~
- PH2: renamed from J2; value PH2 -> ~
- PH3: renamed from J3; value PH3 -> ~
- VBAT: renamed from J16; value VBAT -> ~
- moved S 2.42 mm to (117.6, 56.1)
- moved C5 1.14 mm to (111.6, 82.0)
- renumbered J25 to E, J24 to S, J23 to S, J21 to USART1
Connections:
- net /Pb10 renamed /PB10
Routing:
- net /PB4: track 5.85 -> 57.8 mm, vias 0 -> 1
- net /PB5: track 7.78 -> 42.8 mm, vias 0 -> 4
- net /PA8: track 61.1 -> 29.9 mm, vias 1 -> 3
- net GND: track 198.3 -> 225.0 mm, vias 2 -> 3
- net /PB3: track 6.39 -> 30.0 mm, vias 0 -> 2
- net /PA15: track 20.8 -> 42.1 mm
- net +3.3V: track 135.6 -> 154.4 mm, vias 4 -> 5
- net /USART2RX: track 69.6 -> 66.1 mm
- net /CAN1TX: track 21.4 -> 24.1 mm
- net /CAN2STB: track 6.04 -> 3.82 mm
- net /USART2TX: track 77.9 -> 80.0 mm
- net /CAN1RX: track 24.3 -> 22.2 mm, vias 6 -> 4
- net /USART1RX: track 62.9 -> 60.9 mm
- net /PB2: track 53.3 -> 51.4 mm
- net /CAN2TX: track 18.0 -> 16.6 mm
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Other:
- board outline added: 62.5 x 46.3 mm
