File: sch/adapter/adapter.kicad_sch (KiCad schematic)
At the start: 58 parts, among them J17 CAN2, J18 CAN1, J19 PA0-7, J20 PA8-16, J21 USART1, J22 USART2, J26 RS485, J27 PWR1, J28 PWR2, J29 POWER, SW1 RESET, U1 AT32F435-lqfp48, U2 TJA1049T, U3 TJA1049T, U4 MAX485E, U5 AMS1117-3.3, Y1 8.0 MHz

Commit message: Preparing SilkScreen
Parts:
- added C11: 100n, Capacitor_SMD:C_0805_2012Metric, symbol Device:C
- added U6: W25Q32JVSS, Package_SO:SOIC-8_5.23x5.23mm_P1.27mm, symbol Memory_Flash:W25Q32JVSS
- renumbered J25 to E, J7 to PB0, J8 to PB1, J14 to PB10, J15 to PB11, J1 to PB2, J9 to PB3, J11 to PB4, J10 to PB5, J12 to PB6, J13 to PB7, J4 to PC13, J5 to PC14, J6 to PC15, J2 to PH2, J3 to PH3, J27 to PWR1, J28 to PWR2, J23 to S, J24 to S, J21 to USART1, J16 to VBAT
Connections:
- net +3.3V: now also C11.1, U6.3 (IO2), U6.7 (IO3), U6.8 (VCC)
- net GND: now also C11.2, U6.4 (GND)
- net PA15: now also U6.1 (~{CS})
- net PB3: now also U6.6 (CLK)
- net PB4: now also U6.2 (DO(IO1))
- net PB5: now also U6.5 (DI(IO0))
- net Pb10 renamed PB10
